File: tiny-scarab.kicad_sch (KiCad schematic)
At the start: 28 parts, among them J3 Conn_02x07_Odd_Even, J4 Conn_02x07_Odd_Even, J5 Screw_Hole, J6 Screw_Hole, J7 Screw_Hole, J8 Screw_Hole

Commit message: Change J3 and J4 part numbers
Parts:
- J3, J4: JLCPCB Part # (none) -> C84004; MPN 10129383-914001ALF -> C84004; Manufacturer Amphenol ICC (FCI) -> BOOMELE(Boom Precision Elec); SPN 10129383-914001ALF-ND -> (none); Supplier DigiKey -> (none)
Changed lines of the file:
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@@
       (effects (font (size 1.27 1.27)) hide)
     )
-    (property "Datasheet" "https://cdn.amphenol-cs.com/media/wysiwyg/files/drawing/10129383.pdf" (at 163.83 34.29 0)
-      (effects (font (size 1.27 1.27)) hide)
-    )
-    (property "Manufacturer" "Amphenol ICC (FCI)" (at 165.1 36.83 0)
-      (effects (font (size 1.27 1.27)) hide)
-    )
-    (property "MPN" "10129383-914001ALF" (at 165.1 39.37 0)
-      (effects (font (size 1.27 1.27)) hide)
-    )
-    (property "Supplier" "DigiKey" (at 165.1 41.91 0)
-      (effects (font (size 1.27 1.27)) hide)
-    )
-    (property "SPN" "10129383-914001ALF-ND" (at 165.1 44.45 0)
+    (property "Datasheet" "" (at 163.83 34.29 0)
+      (effects (font (size 1.27 1.27)) hide)
+    )
+    (property "Manufacturer" "BOOMELE(Boom Precision Elec)" (at 165.1 36.83 0)
+      (effects (font (size 1.27 1.27)) hide)
+    )
+    (property "MPN" "C84004" (at 165.1 39.37 0)
+      (effects (font (size 1.27 1.27)) hide)
+    )
+    (property "JLCPCB Part #" "C84004" (at 165.1 44.45 0)
       (effects (font (size 1.27 1.27)) hide)
     )
@@
       (effects (font (size 1.27 1.27)) hide)
     )
-    (property "Datasheet" "https://cdn.amphenol-cs.com/media/wysiwyg/files/drawing/10129383.pdf" (at 163.83 10.16 0)
-      (effects (font (size 1.27 1.27)) hide)
-    )
-    (property "Manufacturer" "Amphenol ICC (FCI)" (at 165.1 12.7 0)
-      (effects (font (size 1.27 1.27)) hide)
-    )
-    (property "MPN" "10129383-914001ALF" (at 165.1 15.24 0)
-      (effects (font (size 1.27 1.27)) hide)
-    )
-    (property "Supplier" "DigiKey" (at 165.1 17.78 0)
-      (effects (font (size 1.27 1.27)) hide)
-    )
-    (property "SPN" "10129383-914001ALF-ND" (at 165.1 20.32 0)
-      (effects (font (size 1.27 1.27)) hide)
-    )
+    (property "Datasheet" "" (at 163.83 10.16 0)
+      (effects (font (size 1.27 1.27)) hide)
+    )
+    (property "Manufacturer" "BOOMELE(Boom Precision Elec)" (at 165.1 12.7 0)
+      (effects (font (size 1.27 1.27)) hide)
+    )
+    (property "MPN" "C84004" (at 165.1 15.24 0)
+      (effects (font (size 1.27 1.27)) hide)
+    )
+    (property "JLCPCB Part #" "C84004" (at 165.1 40.64 0)
+      (effects (font (size 1.27 1.27)) hide)
+    )

Commit message: Change silkscreen
Parts:
- J3, J4: MPN C84004 -> 10129383-914001ALF; Manufacturer BOOMELE(Boom Precision Elec) -> Amphenol ICC (FCI); SPN (none) -> 10129383-914001ALF-ND; Supplier (none) -> DigiKey
Changed lines of the file:
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@@
       (effects (font (size 1.27 1.27)) hide)
     )
-    (property "Datasheet" "" (at 163.83 34.29 0)
-      (effects (font (size 1.27 1.27)) hide)
-    )
-    (property "Manufacturer" "BOOMELE(Boom Precision Elec)" (at 165.1 36.83 0)
-      (effects (font (size 1.27 1.27)) hide)
-    )
-    (property "MPN" "C84004" (at 165.1 39.37 0)
+    (property "Datasheet" "https://cdn.amphenol-cs.com/media/wysiwyg/files/drawing/10129383.pdf" (at 163.83 34.29 0)
+      (effects (font (size 1.27 1.27)) hide)
+    )
+    (property "Manufacturer" "Amphenol ICC (FCI)" (at 165.1 36.83 0)
+      (effects (font (size 1.27 1.27)) hide)
+    )
+    (property "MPN" "10129383-914001ALF" (at 165.1 39.37 0)
       (effects (font (size 1.27 1.27)) hide)
     )
     (property "JLCPCB Part #" "C84004" (at 165.1 44.45 0)
+      (effects (font (size 1.27 1.27)) hide)
+    )
+    (property "Supplier" "DigiKey" (at 165.1 41.91 0)
+      (effects (font (size 1.27 1.27)) hide)
+    )
+    (property "SPN" "10129383-914001ALF-ND" (at 165.1 44.45 0)
       (effects (font (size 1.27 1.27)) hide)
     )
@@
       (effects (font (size 1.27 1.27)) hide)
     )
-    (property "Datasheet" "" (at 163.83 10.16 0)
-      (effects (font (size 1.27 1.27)) hide)
-    )
-    (property "Manufacturer" "BOOMELE(Boom Precision Elec)" (at 165.1 12.7 0)
-      (effects (font (size 1.27 1.27)) hide)
-    )
-    (property "MPN" "C84004" (at 165.1 15.24 0)
+    (property "Datasheet" "https://cdn.amphenol-cs.com/media/wysiwyg/files/drawing/10129383.pdf" (at 163.83 10.16 0)
+      (effects (font (size 1.27 1.27)) hide)
+    )
+    (property "Manufacturer" "Amphenol ICC (FCI)" (at 165.1 12.7 0)
+      (effects (font (size 1.27 1.27)) hide)
+    )
+    (property "MPN" "10129383-914001ALF" (at 165.1 15.24 0)
       (effects (font (size 1.27 1.27)) hide)
     )
@@
       (effects (font (size 1.27 1.27)) hide)
     )
+    (property "Supplier" "DigiKey" (at 165.1 17.78 0)
+      (effects (font (size 1.27 1.27)) hide)
+    )
+    (property "SPN" "10129383-914001ALF-ND" (at 165.1 20.32 0)
+      (effects (font (size 1.27 1.27)) hide)
+    )
